File: hardware/adapters/atari-9pin/chipbridge-atari2600-9pin.kicad_sch (KiCad schematic)
At the start: 1 part, among them J1 AudioJack3_SwitchTR

Commit message: Add hardware bill of materials
Parts:
- J1: MPN (none) -> SJ1-3525N; Manufacturer (none) -> Same Sky
Changed lines of the file:
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@@
 			)
 		)
-		(property "Datasheet" ""
+		(property "Datasheet" "https://www.sameskydevices.com/product/resource/sj1-352xn.pdf"
 			(at 68.58 62.23 0)
 			(hide yes)
@@
 			)
 		)
+		(property "MPN" "SJ1-3525N" (at 0 0 0)
+			(effects
+				(font
+					(size 1.27 1.27)
+				)
+				(hide yes)
+			)
+		)
+		(property "Manufacturer" "Same Sky" (at 0 0 0)
+			(effects
+				(font
+					(size 1.27 1.27)
+				)
+				(hide yes)
+			)
+		)
