File: hardware/adapters/game-gear/chipbridge-gg.kicad_sch (KiCad schematic)
At the start: 2 parts, among them J1 Conn_01x03_Pin, J2 AudioJack3_SwitchTR

Commit message: Add hardware bill of materials
Parts:
- J1: BOM Comments (none) -> Generic 1x3 vertical through-hole pin header, 2.54 mm pitch
- J2: MPN (none) -> SJ1-3525N; Manufacturer (none) -> Same Sky
Changed lines of the file:
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@@
 			)
 		)
-		(property "Datasheet" ""
+		(property "Datasheet" "https://www.sameskydevices.com/product/resource/sj1-352xn.pdf"
 			(at 85.09 67.31 0)
 			(hide yes)
@@
 					(size 1.27 1.27)
 				)
+			)
+		)
+		(property "MPN" "SJ1-3525N" (at 0 0 0)
+			(effects
+				(font
+					(size 1.27 1.27)
+				)
+				(hide yes)
+			)
+		)
+		(property "Manufacturer" "Same Sky" (at 0 0 0)
+			(effects
+				(font
+					(size 1.27 1.27)
+				)
+				(hide yes)
 			)
 		)
@@
 			)
 		)
+		(property "BOM Comments" "Generic 1x3 vertical through-hole pin header, 2.54 mm pitch" (at 0 0 0)
+			(effects
+				(font
+					(size 1.27 1.27)
+				)
+				(hide yes)
+			)
+		)
