File: hardware/main/chipbridge.kicad_sch (KiCad schematic)
At the start: 14 parts, among them J1 CONSOLE_DATA, J2 TRS_MIDI_IN, U1 RP2040-ZERO, U2 6N138

Commit message: Add hardware bill of materials
Parts:
- C1: BOM Comments (none) -> Generic 100 nF ceramic capacitor, 16 V minimum, 2.50 mm lea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
- D1, D2: MF (none) -> Vishay; MP (none) -> BAT46-TAP
- D3: MF (none) -> onsemi; MP (none) -> 1N4148
- D4: BOM Comments (none) -> Generic 3 mm through-hole indicator LED; observe polarity
- J1, J2: MF (none) -> Same Sky; MP (none) -> SJ1-3525N
- R1, R2, R4, R5: BOM Comments (none) -> Generic 470 ohm axial resistor, 0.25 W or greater, DIN0204 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
- R3: BOM Comments (none) -> Generic 220 ohm axial resistor, 0.25 W or greater, DIN0204 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
- U2: BOM Comments (none) -> 8-pin DIP optocoupler; a DIP-8 socket is optional and is no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; MF (none) -> onsemi; MP (none) -> 6N138M
Changed lines of the file:
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@@
+			)
+		)
+		(property "BOM Comments" "Generic 470 ohm axial resistor, 0.25 W or greater, DIN0204 body" (at 0 0 0)
+			(effects
+				(font
+					(size 1.27 1.27)
+				)
+				(hide yes)
 			)
 		)
@@
 			)
 		)
+		(property "BOM Comments" "Generic 100 nF ceramic capacitor, 16 V minimum, 2.50 mm lead pitch, body no larger than footprint" (at 0 0 0)
+			(effects
+				(font
+					(size 1.27 1.27)
+				)
+				(hide yes)
+			)
+		)
 		(pin "1"
 		)
@@
 			)
 		)
+		(property "BOM Comments" "Generic 470 ohm axial resistor, 0.25 W or greater, DIN0204 body" (at 0 0 0)
+			(effects
+				(font
+					(size 1.27 1.27)
+				)
+				(hide yes)
+			)
+		)
 		(pin "2"
 		)
@@
 			)
 		)
-		(property "Datasheet" "http://www.onsemi.com/pub/Collateral/HCPL2731-D.pdf"
+		(property "Datasheet" "https://www.onsemi.com/download/data-sheet/pdf/hcpl2731m-d.pdf"
 			(at 197.104 78.74 0)
 			(hide yes)
@@
 					(size 1.27 1.27)
 				)
+			)
+		)
+		(property "BOM Comments" "8-pin DIP optocoupler; a DIP-8 socket is optional and is not included in this BOM" (at 0 0 0)
+			(effects
+				(font
+					(size 1.27 1.27)
+				)
+				(hide yes)
+			)
+		)
+		(property "MP" "6N138M" (at 0 0 0)
+			(effects
+				(font
+					(size 1.27 1.27)
+				)
+				(hide yes)
+			)
+		)
+		(property "MF" "onsemi" (at 0 0 0)
+			(effects
+				(font
+					(size 1.27 1.27)
+				)
+				(hide yes)
 			)
 		)
@@
 			)
 		)
-		(property "Datasheet" "http://www.vishay.com/docs/85662/bat46.pdf"
+		(property "Datasheet" "https://www.vishay.com/docs/85662/bat46.pdf"
 			(at 68.58 50.8 0)
 			(hide yes)
@@
 					(size 1.27 1.27)
 				)
+			)
+		)
+		(property "MP" "BAT46-TAP" (at 0 0 0)
+			(effects
+				(font
+					(size 1.27 1.27)
+				)
+				(hide yes)
+			)
+		)
+		(property "MF" "Vishay" (at 0 0 0)
+			(effects
+				(font
+					(size 1.27 1.27)
+				)
+				(hide yes)
 			)
 		)
@@
 			)
 		)
-		(property "Datasheet" "Connector_Audio:Jack_3.5mm_CUI_SJ1-3525N_Horizontal"
+		(property "Datasheet" "https://www.sameskydevices.com/product/resource/sj1-352xn.pdf"
 			(at 137.922 43.688 0)
 			(hide yes)
@@
 					(size 1.27 1.27)
 				)
+			)
+		)
+		(property "MP" "SJ1-3525N" (at 0 0 0)
+			(effects
+				(font
+					(size 1.27 1.27)
+				)
+				(hide yes)
+			)
+		)
+		(property "MF" "Same Sky" (at 0 0 0)
+			(effects
+				(font
+					(size 1.27 1.27)
+				)
+				(hide yes)
 			)
 		)
@@
 			)
 		)
-		(property "Datasheet" ""
+		(property "Datasheet" "https://www.waveshare.com/wiki/RP2040-Zero"
 			(at 91.44 64.77 0)
 			(hide yes)
@@
 			)
 		)
-		(property "Datasheet" ""
+		(property "Datasheet" "https://www.sameskydevices.com/product/resource/sj1-352xn.pdf"
 			(at 138.176 66.04 0)
 			(hide yes)
@@
 					(size 1.27 1.27)
 				)
+			)
+		)
+		(property "MP" "SJ1-3525N" (at 0 0 0)
+			(effects
+				(font
+					(size 1.27 1.27)
+				)
+				(hide yes)
+			)
+		)
+		(property "MF" "Same Sky" (at 0 0 0)
+			(effects
+				(font
+					(size 1.27 1.27)
+				)
+				(hide yes)
 			)
 		)
@@
 			)
 		)
-		(property "Datasheet" "http://www.vishay.com/docs/85662/bat46.pdf"
+		(property "Datasheet" "https://www.vishay.com/docs/85662/bat46.pdf"
 			(at 36.83 53.34 0)
 			(hide yes)
@@
 					(size 1.27 1.27)
 				)
+			)
+		)
+		(property "MP" "BAT46-TAP" (at 0 0 0)
+			(effects
+				(font
+					(size 1.27 1.27)
+				)
+				(hide yes)
+			)
+		)
+		(property "MF" "Vishay" (at 0 0 0)
+			(effects
+				(font
+					(size 1.27 1.27)
+				)
+				(hide yes)
 			)
 		)
@@
 			)
 		)
+		(property "BOM Comments" "Generic 470 ohm axial resistor, 0.25 W or greater, DIN0204 body" (at 0 0 0)
+			(effects
+				(font
+					(size 1.27 1.27)
+				)
+				(hide yes)
+			)
+		)
 		(pin "1"
 		)
@@
 			)
 		)
-		(property "Datasheet" "https://assets.nexperia.com/documents/data-sheet/1N4148_1N4448.pdf"
+		(property "Datasheet" "https://www.onsemi.com/pdf/datasheet/1n914-d.pdf"
 			(at 171.45 72.39 0)
 			(hide yes)
@@
 					(size 1.27 1.27)
 				)
+			)
+		)
+		(property "MP" "1N4148" (at 0 0 0)
+			(effects
+				(font
+					(size 1.27 1.27)
+				)
+				(hide yes)
+			)
+		)
+		(property "MF" "onsemi" (at 0 0 0)
+			(effects
+				(font
+					(size 1.27 1.27)
+				)
+				(hide yes)
 			)
 		)
@@
 			)
 		)
+		(property "BOM Comments" "Generic 220 ohm axial resistor, 0.25 W or greater, DIN0204 body" (at 0 0 0)
+			(effects
+				(font
+					(size 1.27 1.27)
+				)
+				(hide yes)
+			)
+		)
 		(pin "1"
 		)
@@
 			)
 		)
+		(property "BOM Comments" "Generic 470 ohm axial resistor, 0.25 W or greater, DIN0204 body" (at 0 0 0)
+			(effects
+				(font
+					(size 1.27 1.27)
+				)
+				(hide yes)
+			)
+		)
 		(pin "1"
 		)
@@
 			)
 		)
+		(property "BOM Comments" "Generic 3 mm through-hole indicator LED; observe polarity" (at 0 0 0)
+			(effects
+				(font
+					(size 1.27 1.27)
+				)
+				(hide yes)
+			)
+		)
